Commit message: Add simple box/cylinder <visual> geometry to the vehicle URDF
Purely cosmetic addition to the step-3 URDF, doesn't touch the
<ros2_control> block or joint structure at all: a chassis box and four
wheel cylinders, using simple_vehicle.py's actual dimensions/colors
(CHASSIS_DIMS=2.6x1.6x0.4 at chassis_z=1.19 -- WHEEL_RADIUS+
SUSPENSION_TRAVEL_REST+CHASSIS_CG_HEIGHT, not an arbitrary number --
red chassis, dark wheels) instead of arbitrary placeholder shapes. No
<inertial>/<collision> -- this URDF isn't used to run physics (Chrono
does that inside the FMU), just for RViz display and ros2_control's
joint/interface bookkeeping.

Hit the same "--" inside XML comments issue as step 3's original
commits and fixed it the same way (em dash).

Verified by actually re-running the display launch file and
screenshotting RViz: a red chassis box sits correctly above four dark
wheel cylinders at the right positions, Global Status: Ok.

Co-Authored-By: Claude Sonnet 5 <noreply@anthropic.com>
Claude-Session: https://claude.ai/code/session_01UULNnKKARJpjHeGbdgzYdT

File: ros2_control/urdf/chrono_vehicle.urdf (robot description, URDF)
Before this commit: robot chrono_vehicle, 5 links, 4 joints
Links:
- link base_link: geometry visual box size=2.6 1.6 0.4
- link front_left_wheel: geometry visual cylinder length=0.22 radius=0.32
- link front_right_wheel: geometry visual cylinder length=0.22 radius=0.32
- link rear_left_wheel: geometry visual cylinder length=0.22 radius=0.32
- link rear_right_wheel: geometry visual cylinder length=0.22 radius=0.32

Commit message: Add front wheel spin joints so 4WD's front-axle motion is actually visible
User noticed chrono_fmu_system_interface_check's output only ever
showed rear_left/right_wheel_joint/velocity, even with 4WD on, and
asked why. Root cause: the URDF never had a joint representing front
wheel spin at all -- it was designed rear-drive-only (step 3), so
front wheels only got a steering (position) joint. 4WD's effect was
only visible indirectly, through the shared speed_mps-derived
"rear wheel velocity" changing when the front axle also started
contributing torque.

URDF change (both chrono_vehicle.urdf and chrono_vehicle_split.urdf):
added front_left/right_knuckle links between the existing steering
revolute and a new front_left/right_wheel_joint (continuous, velocity)
-- a single link can't be the child of two independent joints, so the
knuckle is needed as a pass-through, matching vehicle_native.cpp's own
body chain (upright -> knuckle -> wheel) rather than inventing a
different structure. The new joints are declared with a
state_interface only, no command_interface: ackermann_steering_controller
has no front-traction command path at all, and 4WD's torque is
already driven from the rear-axle command's P-loop, so nothing should
ever write to these. Hit the recurring "--" inside an XML comment
issue a 4th time, same em-dash fix.

Plugin changes (ChronoFmuSystemInterface and ChronoEcuBridgeSystemInterface,
both need this since the same URDF works for both): on_init()'s joint
validation relaxed from "exactly 1 command_interface" to "0 or 1"
(state_interface stays required at exactly 1), tracked via a new
JointIO::has_command field. export_command_interfaces() skips
has_command=false joints. Caught and avoided a real bug before it
happened: write()'s rear-wheel command-averaging loop was keyed only
on interface==VELOCITY, which would have silently pulled in the new
front joints' meaningless default-0.0 .command and diluted the P
loop's actual target -- added the has_command check to that loop too.
read() needed no change at all: it already treats every
HW_IF_VELOCITY joint uniformly, so front wheel state got picked up
for free.

Verified: chrono_fmu_system_interface_check now exports 6 state / 4
command interfaces, with front_left/right_wheel_joint/velocity
reporting the same value as the rear joints (same no-slip
approximation, expected) -- and the rear joints' own numbers are
bit-identical to before this change, confirming this is purely
additive visibility with zero logic change. Split version re-verified
live: idle stays bounded (0.0338 rad/s), linear.x=1.0/angular.z=0.3
converges smoothly with all four velocity joints (front+rear,
left+right) reporting the same value (2.2445 rad/s).

Co-Authored-By: Claude Sonnet 5 <noreply@anthropic.com>
Claude-Session: https://claude.ai/code/session_01UULNnKKARJpjHeGbdgzYdT

File: ros2_control/urdf/chrono_vehicle.urdf (robot description, URDF)
Before this commit: robot chrono_vehicle, 5 links, 4 joints
Links:
- added link front_left_knuckle
- added link front_right_knuckle
Joints:
- added joint front_left_wheel_joint: type continuous, parent front_left_knuckle, child front_left_wheel, origin xyz=0 0 0 rpy=0 0 0, axis 0 1 0
- added joint front_right_wheel_joint: type continuous, parent front_right_knuckle, child front_right_wheel, origin xyz=0 0 0 rpy=0 0 0, axis 0 1 0
- joint front_left_steering_joint: child front_left_wheel -> front_left_knuckle
- joint front_right_steering_joint: child front_right_wheel -> front_right_knuckle

File: ros2_control/urdf/chrono_vehicle_split.urdf (robot description, URDF)
Before this commit: robot chrono_vehicle_split, 5 links, 4 joints
Links:
- added link front_left_knuckle
- added link front_right_knuckle
Joints:
- added joint front_left_wheel_joint: type continuous, parent front_left_knuckle, child front_left_wheel, origin xyz=0 0 0 rpy=0 0 0, axis 0 1 0
- added joint front_right_wheel_joint: type continuous, parent front_right_knuckle, child front_right_wheel, origin xyz=0 0 0 rpy=0 0 0, axis 0 1 0
- joint front_left_steering_joint: child front_left_wheel -> front_left_knuckle
- joint front_right_steering_joint: child front_right_wheel -> front_right_knuckle

Commit message: Make the FMU-driven robot actually visible/moving in RViz -- 4 real gaps found and fixed live, both tracks
Opening the 6x6 build in RViz against a real running controller_manager
(not display.launch.py's fake joint_state_publisher_gui sliders) was the
first time anyone had visualized the real FMU-driven robot -- it exposed
four separate, real gaps, each found live and fixed in turn:

1. All 6 wheels failed to render ("No transform from [wheel] to
   [base_link]"). Wheel joints only ever exported a velocity
   state_interface (the FMU has no per-wheel angle), but
   robot_state_publisher needs a numeric position for every non-fixed
   joint's TF, even continuous ones -- position came through as NaN.
   Not 6x6-specific; the same gap existed since the 4WD front-spin-joint
   work, just never noticed. Fixed with a dead-reckoned
   JointIO::dead_reckoned_position (visualization-only, integrated from
   velocity each read(), never fed back into control) on both
   ChronoFmuSystemInterface and ChronoEcuBridgeSystemInterface, exported
   as an additional position state_interface. on_init()'s joint
   validation rewritten accordingly (position-type: exactly 1
   state_interface; velocity-type: exactly 2, velocity+position -- must
   match what's actually exported or resource_manager errors). All 4
   URDFs updated to declare the extra state_interface.

2. Wheels rendered but never appeared to spin -- a plain <cylinder> is
   rotationally symmetric about its own axis, so the dead-reckoned
   position updates the TF correctly but is visually imperceptible.
   Added a small off-axis <box> stripe per wheel.

3. The stripe rendered solid black instead of its intended silver --
   RViz/Ogre only honors the FIRST <visual>'s material when a link has
   multiple <visual> elements (confirmed live: rotation was already
   correct, only the color was wrong; URDF material name/reference were
   fine). Fixed by giving the stripe its own separate link + fixed joint
   to the wheel instead of a second <visual> in the same link -- a fixed
   joint needs no <ros2_control> entry and is published as static TF
   automatically.

4. Wheels spun correctly but the chassis never appeared to move -- RViz's
   Fixed Frame was saved as base_link (definitionally motionless when
   selected as the fixed frame). Switching to odom failed too because no
   odom frame ever appeared on /tf, even though
   ackermann_steering_controller's enable_odom_tf defaults to true and
   /ackermann_steering_controller/odometry + tf_odometry were both
   publishing correct, growing odom->base_link data at 500Hz -- the
   transform only ever went to the controller's own private namespaced
   topic (~/tf_odometry), never to the global /tf RViz subscribes to.
   spawner has no per-controller remap flag in Humble, so the fix lives
   on ros2_control_node itself: remapped
   /ackermann_steering_controller/tf_odometry to /tf in both launch
   files (message types match exactly, both tf2_msgs/TFMessage).

Colors refreshed while at it, per request: chassis_red -> deep crimson,
wheel_dark -> graphite, new wheel_marker -> silver.

Verified: chrono_fmu_system_interface_check bit-exact unchanged on both
4-wheel (3.637180) and 6x6 (2.709956) velocity -- the position export is
purely additive, zero control-path impact; the new position field grows
correctly. Live in the user's own RViz, both tracks (in-process and
split): no transform errors, all wheels render and visibly spin with the
correct color, chassis actually translates with Fixed Frame=odom.

Co-Authored-By: Claude Sonnet 5 <noreply@anthropic.com>
Claude-Session: https://claude.ai/code/session_01UULNnKKARJpjHeGbdgzYdT

File: ros2_control/urdf/chrono_vehicle.urdf (robot description, URDF)
Before this commit: robot chrono_vehicle, 7 links, 6 joints
Links:
- added link front_left_wheel_marker; visual box size=0.22 0.015 0.04
- added link front_right_wheel_marker; visual box size=0.22 0.015 0.04
- added link rear_left_wheel_marker; visual box size=0.22 0.015 0.04
- added link rear_right_wheel_marker; visual box size=0.22 0.015 0.04
Joints:
- added joint front_left_wheel_marker_joint: type fixed, parent front_left_wheel, child front_left_wheel_marker, origin xyz=0.15 0.115 0 rpy=0 0 0
- added joint front_right_wheel_marker_joint: type fixed, parent front_right_wheel, child front_right_wheel_marker, origin xyz=0.15 -0.115 0 rpy=0 0 0
- added joint rear_left_wheel_marker_joint: type fixed, parent rear_left_wheel, child rear_left_wheel_marker, origin xyz=0.15 0.115 0 rpy=0 0 0
- added joint rear_right_wheel_marker_joint: type fixed, parent rear_right_wheel, child rear_right_wheel_marker, origin xyz=0.15 -0.115 0 rpy=0 0 0

File: ros2_control/urdf/chrono_vehicle_6x6.urdf (robot description, URDF)
Before this commit: robot chrono_vehicle_6x6, 9 links, 8 joints
Links:
- added link front_left_wheel_marker; visual box size=0.22 0.015 0.04
- added link front_right_wheel_marker; visual box size=0.22 0.015 0.04
- added link mid_left_wheel_marker; visual box size=0.22 0.015 0.04
- added link mid_right_wheel_marker; visual box size=0.22 0.015 0.04
- added link rear_left_wheel_marker; visual box size=0.22 0.015 0.04
- added link rear_right_wheel_marker; visual box size=0.22 0.015 0.04
Joints:
- added joint front_left_wheel_marker_joint: type fixed, parent front_left_wheel, child front_left_wheel_marker, origin xyz=0.15 0.115 0 rpy=0 0 0
- added joint front_right_wheel_marker_joint: type fixed, parent front_right_wheel, child front_right_wheel_marker, origin xyz=0.15 -0.115 0 rpy=0 0 0
- added joint mid_left_wheel_marker_joint: type fixed, parent mid_left_wheel, child mid_left_wheel_marker, origin xyz=0.15 0.115 0 rpy=0 0 0
- added joint mid_right_wheel_marker_joint: type fixed, parent mid_right_wheel, child mid_right_wheel_marker, origin xyz=0.15 -0.115 0 rpy=0 0 0
- added joint rear_left_wheel_marker_joint: type fixed, parent rear_left_wheel, child rear_left_wheel_marker, origin xyz=0.15 0.115 0 rpy=0 0 0
- added joint rear_right_wheel_marker_joint: type fixed, parent rear_right_wheel, child rear_right_wheel_marker, origin xyz=0.15 -0.115 0 rpy=0 0 0

File: ros2_control/urdf/chrono_vehicle_split.urdf (robot description, URDF)
Before this commit: robot chrono_vehicle_split, 7 links, 6 joints
Links:
- added link front_left_wheel_marker; visual box size=0.22 0.015 0.04
- added link front_right_wheel_marker; visual box size=0.22 0.015 0.04
- added link rear_left_wheel_marker; visual box size=0.22 0.015 0.04
- added link rear_right_wheel_marker; visual box size=0.22 0.015 0.04
Joints:
- added joint front_left_wheel_marker_joint: type fixed, parent front_left_wheel, child front_left_wheel_marker, origin xyz=0.15 0.115 0 rpy=0 0 0
- added joint front_right_wheel_marker_joint: type fixed, parent front_right_wheel, child front_right_wheel_marker, origin xyz=0.15 -0.115 0 rpy=0 0 0
- added joint rear_left_wheel_marker_joint: type fixed, parent rear_left_wheel, child rear_left_wheel_marker, origin xyz=0.15 0.115 0 rpy=0 0 0
- added joint rear_right_wheel_marker_joint: type fixed, parent rear_right_wheel, child rear_right_wheel_marker, origin xyz=0.15 -0.115 0 rpy=0 0 0

File: ros2_control/urdf/chrono_vehicle_split_6x6.urdf (robot description, URDF)
Before this commit: robot chrono_vehicle_split_6x6, 9 links, 8 joints
Links:
- added link front_left_wheel_marker; visual box size=0.22 0.015 0.04
- added link front_right_wheel_marker; visual box size=0.22 0.015 0.04
- added link mid_left_wheel_marker; visual box size=0.22 0.015 0.04
- added link mid_right_wheel_marker; visual box size=0.22 0.015 0.04
- added link rear_left_wheel_marker; visual box size=0.22 0.015 0.04
- added link rear_right_wheel_marker; visual box size=0.22 0.015 0.04
Joints:
- added joint front_left_wheel_marker_joint: type fixed, parent front_left_wheel, child front_left_wheel_marker, origin xyz=0.15 0.115 0 rpy=0 0 0
- added joint front_right_wheel_marker_joint: type fixed, parent front_right_wheel, child front_right_wheel_marker, origin xyz=0.15 -0.115 0 rpy=0 0 0
- added joint mid_left_wheel_marker_joint: type fixed, parent mid_left_wheel, child mid_left_wheel_marker, origin xyz=0.15 0.115 0 rpy=0 0 0
- added joint mid_right_wheel_marker_joint: type fixed, parent mid_right_wheel, child mid_right_wheel_marker, origin xyz=0.15 -0.115 0 rpy=0 0 0
- added joint rear_left_wheel_marker_joint: type fixed, parent rear_left_wheel, child rear_left_wheel_marker, origin xyz=0.15 0.115 0 rpy=0 0 0
- added joint rear_right_wheel_marker_joint: type fixed, parent rear_right_wheel, child rear_right_wheel_marker, origin xyz=0.15 -0.115 0 rpy=0 0 0
